Commit message: Simulation updates

File: ROS/osr_gazebo/urdf/osr.urdf.xacro (robot description, xacro)
@@ -417,5 +417,5 @@
             <parent link="base_link"/>
             <child link="imu_link"/>
-            <origin xyz="0 0 0" rpy="0 0 0"/>
+            <origin xyz="0.035 0.065 0" rpy="0 0 0"/>
         </joint>
     <link name="imu_link"></link>
@@ -427,5 +427,5 @@
     <link name="lidar_link">
         <visual>
-            <geometry><cylinder radius="0.081" length="0.04"/></geometry>
+            <geometry><cylinder radius="0.0405" length="0.04"/></geometry>
         </visual>
     </link>
@@ -433,24 +433,86 @@
         <sensor name="lidar" type="gpu_lidar">
             <gz_frame_id>lidar_link</gz_frame_id>
-            <topic>/lidar</topic>
+            <topic>/scan</topic>
             <pose>0 0 0 0 0 0</pose>
             <always_on>true</always_on>
             <visualize>true</visualize>
             <update_rate>10</update_rate>
-            <ray>
-            <scan>
-                <horizontal>
-                <samples>32000</samples>
-                <resolution>1</resolution>
-                <min_angle>-3.14</min_angle>
-                <max_angle>3.14</max_angle>
-                </horizontal>
-            </scan>
-            <range>
-                <min>0.05</min>
-                <max>18.0</max>
-            </range>
-            </ray>
+            <lidar>
+                <scan>
+                    <horizontal>
+                    <samples>720</samples>
+                    <resolution>1</resolution>
+                    <min_angle>-3.14</min_angle>
+                    <max_angle>3.14</max_angle>
+                    </horizontal>
+                </scan>
+                <range>
+                    <min>0.05</min>
+                    <max>18.0</max>
+                </range>
+            </lidar>
         </sensor>
+    </gazebo>
+    <gazebo reference="imu_link">
+    <sensor name="imu_sensor" type="imu">
+        <always_on>true</always_on>
+        <update_rate>100</update_rate>
+        <visualize>true</visualize>
+        <topic>/imu</topic>
+        <imu>
+        <angular_velocity>
+            <x>
+            <noise type="gaussian">
+                <mean>0.0</mean>
+                <stddev>2e-4</stddev>
+                <bias_mean>0.0000075</bias_mean>
+                <bias_stddev>0.0000008</bias_stddev>
+            </noise>
+            </x>
+            <y>
+            <noise type="gaussian">
+                <mean>0.0</mean>
+                <stddev>2e-4</stddev>
+                <bias_mean>0.0000075</bias_mean>
+                <bias_stddev>0.0000008</bias_stddev>
+            </noise>
+            </y>
+            <z>
+            <noise type="gaussian">
+                <mean>0.0</mean>
+                <stddev>2e-4</stddev>
+                <bias_mean>0.0000075</bias_mean>
+                <bias_stddev>0.0000008</bias_stddev>
+            </noise>
+            </z>
+        </angular_velocity>
+        <linear_acceleration>
+            <x>
+            <noise type="gaussian">
+                <mean>0.0</mean>
+                <stddev>1.7e-2</stddev>
+                <bias_mean>0.1</bias_mean>
+                <bias_stddev>0.001</bias_stddev>
+            </noise>
+            </x>
+            <y>
+            <noise type="gaussian">
+                <mean>0.0</mean>
+                <stddev>1.7e-2</stddev>
+                <bias_mean>0.1</bias_mean>
+                <bias_stddev>0.001</bias_stddev>
+            </noise>
+            </y>
+            <z>
+            <noise type="gaussian">
+                <mean>0.0</mean>
+                <stddev>1.7e-2</stddev>
+                <bias_mean>0.1</bias_mean>
+                <bias_stddev>0.001</bias_stddev>
+            </noise>
+            </z>
+        </linear_acceleration>
+        </imu>
+    </sensor>
     </gazebo>
     <xacro:insert_velocity_transmission name="rear_wheel_joint_right"/>
